File: Hardware/Qwiic_Keyboard_Explorer.brd (EAGLE design)
At the start: 143.5 x 77.5 mm, 75 parts, among them U1 PRO_MICRO_C

Commit message: Proto x01
Parts:
- added U$25: (no value), Labels:GND-04
- added U$26: (no value), buzzard_labels (2):D101
- added U$27: (no value), buzzard_labels (2):D162
- added U$28: (no value), buzzard_labels (2):D143
- added U$29: (no value), buzzard_labels (2):D154
- added U$30: (no value), buzzard_labels (2):TX5
- added U$31: (no value), buzzard_labels (2):RX6
- added U$32: (no value), SparkFun-Aesthetics:OSHW-LOGO-M_COPPER
- U$12: device SparkFun-Hardware:STAND-OFF -> buzzard_labels (2):5V0
- moved U$12 1.27 mm to (40.6, 72.4)
Other:
- board text added: "x01"

Commit message: Aesthetic tweaks to eagle files
Parts:
- FRAME1: value FRAME-LETTERNO_PACKAGE -> FRAME-LEDGER; device SparkFun-Aesthetics:DUMMY -> SparkFun-Aesthetics:CREATIVE_COMMONS
- moved FRAME1 20.7 mm to (20.3, -8.89)
Other:
- board text added: "N.Poole"
Changed lines of the file:
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@@
 <?xml version="1.0" encoding="utf-8"?>
 <!DOCTYPE eagle SYSTEM "eagle.dtd">
-<eagle version="9.5.2">
+<eagle version="9.6.2">
 <drawing>
 <settings>
-<setting alwaysvectorfont="yes"/>
+<setting alwaysvectorfont="no"/>
 <setting verticaltext="up"/>
 </settings>
@@
 <wire x1="0" y1="2.54" x2="2.54" y2="0" width="0.254" layer="49" curve="90"/>
 <wire x1="140.97" y1="0" x2="143.51" y2="2.54" width="0.254" layer="49" curve="90"/>
+<text x="46.99" y="-10.16" size="1.778" layer="51">N.Poole</text>
 </plain>
 <attributes>
@@
 <elements>
 <element name="U1" library="SparkFun-Boards" package="PRO_MICRO_C" value="PRO_MICRO_C" x="16.51" y="60.96" smashed="yes" rot="R90"/>
-<element name="FRAME1" library="SparkFun-Aesthetics" package="DUMMY" value="FRAME-LETTERNO_PACKAGE" x="5.08" y="5.08" smashed="yes">
-<attribute name="DESIGNER" value="Nobody" x="5.08" y="5.08" size="1.778" layer="27" font="vector" ratio="15" display="off"/>
-<attribute name="VERSION" value="v01" x="5.08" y="5.08" size="1.778" layer="27" font="vector" ratio="15" display="off"/>
-</element>
 <element name="S1" library="SparkFun-Switches" package="CHERRY-MX-LED-1U" value="MECHANICAL-KEYBOARD1U" x="5.08" y="24.13" smashed="yes">
 <attribute name="NAME" x="7.62" y="33.655" size="0.6096" layer="25" font="vector" ratio="20" rot="R90" align="bottom-center"/>
@@
 <element name="U$31" library="buzzard_labels (2)" package="RX6" value="" x="35.56" y="54.61" smashed="yes"/>
 <element name="U$32" library="SparkFun-Aesthetics" package="OSHW-LOGO-M_COPPER" value="" x="129.54" y="2.54" smashed="yes" rot="MR0"/>
+<element name="FRAME1" library="SparkFun-Aesthetics" package="CREATIVE_COMMONS" value="FRAME-LEDGER" x="20.32" y="-8.89" smashed="yes">
+<attribute name="DESIGNER" value="" x="20.32" y="-8.89" size="1.778" layer="27" display="off"/>
+<attribute name="REV" value="" x="20.32" y="-8.89" size="1.778" layer="27" display="off"/>
+</element>
 </elements>
 <signals>
