File: Hardware/Qwiic_Keyboard_Explorer.sch (EAGLE design)
At the start: 51 parts, among them U1 PRO_MICRO_C

Commit message: Aesthetic tweaks to eagle files
Parts:
- FRAME1: value FRAME-LETTERNO_PACKAGE -> FRAME-LEDGER; device SparkFun-Aesthetics:FRAME-LETTERNO_PACKAGE -> SparkFun-Aesthetics:FRAME-LEDGER
Other:
- note added: "Keyswitch Matrix"
- note added: "Mode Select Switch"
- note added: "N.Poole"
- note added: "Pro Micro C Header"
- note added: "Prototyping Space"
- moved on the sheet: D1, D10, D11, D12, D13, D14, D2, D3, D4, D5, D6, D7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
